File: RS485-CH340.kicad_pcb (KiCad board)
At the start: 2 copper layers, 22.5 x 14.5 mm, 13 parts, among them J1 USB_A, J2 Conn_01x04_Pin, U1 CH340N, U2 THVD1406DR

Commit message: Update back/front/pcb/schematic.png Generate BOM and convert to .xlxx format Update README.md
Parts:
- C1, C2: footprint Capacitor_SMD:C_0603_1608Metric -> Capacitor_SMD:C_0603_1608Metric_Pad1.08x0.95mm_HandSolder
- D1: value LED -> LED BLU
- D2: value LED -> LED GRN
- R1, R2: footprint Resistor_SMD:R_0603_1608Metric -> Resistor_SMD:R_0603_1608Metric_Pad0.98x0.95mm_HandSolder
Changed lines of the file:
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@@
 			)
 		)
-		(property "Datasheet" "~"
+		(property "Datasheet" "http://cnctech.us/pdfs/1001-011-01101.pdf"
 			(at 0 0 180)
 			(layer "F.Fab")
@@
 		)
 	)
-	(footprint "Resistor_SMD:R_0603_1608Metric"
+	(footprint "Resistor_SMD:R_0603_1608Metric_Pad0.98x0.95mm_HandSolder"
 		(layer "F.Cu")
 		(at 148.082 95.694 90)
-		(descr "Resistor SMD 0603 (1608 Metric), square (rectangular) end terminal, IPC-7351 nominal, (Body size source: IPC-SM-782 page 72, https://www.pcb-3d.com/wordpress/wp-content/uploads/ipc-sm-782a_amendment_1_and_2.pdf)")
-		(tags "resistor")
+		(descr "Resistor SMD 0603 (1608 Metric), square (rectangular) end terminal, IPC-7351 nominal with elongated pad for handsoldering. (Body size source: IPC-SM-782 page 72, https://www.pcb-3d.com/wordpress/wp-content/uploads/ipc-sm-782a_amendment_1_and_2.pdf)")
+		(tags "resistor handsolder")
 		(property "Reference" "R1"
-			(at -1.969 0 90)
+			(at -2.096 0 90)
 			(layer "F.SilkS")
 			(effects
 				(font
-					(size 0.6604 0.6604)
+					(size 0.8 0.8)
 					(thickness 0.15)
 				)
@@
 		(duplicate_pad_numbers_are_jumpers no)
 		(fp_line
-			(start -0.237258 -0.5225)
-			(end 0.237258 -0.5225)
+			(start -0.254724 -0.5225)
+			(end 0.254724 -0.5225)
 			(stroke
 				(width 0.12)
@@
 		)
 		(fp_line
-			(start -0.237258 0.5225)
-			(end 0.237258 0.5225)
+			(start -0.254724 0.5225)
+			(end 0.254724 0.5225)
 			(stroke
 				(width 0.12)
@@
 		)
 		(fp_rect
-			(start -1.48 -0.73)
-			(end 1.48 0.73)
+			(start -1.65 -0.73)
+			(end 1.65 0.73)
 			(stroke
 				(width 0.05)
@@
 		)
 		(pad "1" smd roundrect
-			(at -0.825 0 90)
-			(size 0.8 0.95)
+			(at -0.9125 0 90)
+			(size 0.975 0.95)
 			(layers "F.Cu" "F.Mask" "F.Paste")
 			(roundrect_rratio 0.25)
@@
 		)
 		(pad "2" smd roundrect
-			(at 0.825 0 90)
-			(size 0.8 0.95)
+			(at 0.9125 0 90)
+			(size 0.975 0.95)
 			(layers "F.Cu" "F.Mask" "F.Paste")
 			(roundrect_rratio 0.25)
@@
 		)
 	)
-	(footprint "Capacitor_SMD:C_0603_1608Metric"
+	(footprint "Capacitor_SMD:C_0603_1608Metric_Pad1.08x0.95mm_HandSolder"
 		(layer "F.Cu")
 		(at 149.098 99.949)
-		(descr "Capacitor SMD 0603 (1608 Metric), square (rectangular) end terminal, IPC-7351 nominal, (Body size source: IPC-SM-782 page 76, https://www.pcb-3d.com/wordpress/wp-content/uploads/ipc-sm-782a_amendment_1_and_2.pdf)")
-		(tags "capacitor")
+		(descr "Capacitor SMD 0603 (1608 Metric), square (rectangular) end terminal, IPC-7351 nominal with elongated pad for handsoldering. (Body size source: IPC-SM-782 page 76, https://www.pcb-3d.com/wordpress/wp-content/uploads/ipc-sm-782a_amendment_1_and_2.pdf)")
+		(tags "capacitor handsolder")
 		(property "Reference" "C2"
-			(at 0 -0.762 0)
+			(at 0 -0.889 0)
 			(layer "F.SilkS")
 			(effects
 				(font
-					(size 0.6604 0.6604)
+					(size 0.8 0.8)
 					(thickness 0.15)
 				)
@@
 		(duplicate_pad_numbers_are_jumpers no)
 		(fp_line
-			(start -0.14058 -0.51)
-			(end 0.14058 -0.51)
+			(start -0.146267 -0.51)
+			(end 0.146267 -0.51)
 			(stroke
 				(width 0.12)
@@
 		)
 		(fp_line
-			(start -0.14058 0.51)
-			(end 0.14058 0.51)
+			(start -0.146267 0.51)
+			(end 0.146267 0.51)
 			(stroke
 				(width 0.12)
@@
 		)
 		(fp_rect
-			(start -1.48 -0.73)
-			(end 1.48 0.73)
+			(start -1.65 -0.73)
+			(end 1.65 0.73)
 			(stroke
 				(width 0.05)
@@
 		)
 		(pad "1" smd roundrect
-			(at -0.775 0)
-			(size 0.9 0.95)
+			(at -0.8625 0)
+			(size 1.075 0.95)
 			(layers "F.Cu" "F.Mask" "F.Paste")
 			(roundrect_rratio 0.25)
@@
 		)
 		(pad "2" smd roundrect
-			(at 0.775 0)
-			(size 0.9 0.95)
+			(at 0.8625 0)
+			(size 1.075 0.95)
 			(layers "F.Cu" "F.Mask" "F.Paste")
 			(roundrect_rratio 0.25)
@@
 		)
 	)
-	(footprint "Capacitor_SMD:C_0603_1608Metric"
+	(footprint "Capacitor_SMD:C_0603_1608Metric_Pad1.08x0.95mm_HandSolder"
 		(layer "F.Cu")
 		(at 146.05 99.949 180)
-		(descr "Capacitor SMD 0603 (1608 Metric), square (rectangular) end terminal, IPC-7351 nominal, (Body size source: IPC-SM-782 page 76, https://www.pcb-3d.com/wordpress/wp-content/uploads/ipc-sm-782a_amendment_1_and_2.pdf)")
-		(tags "capacitor")
+		(descr "Capacitor SMD 0603 (1608 Metric), square (rectangular) end terminal, IPC-7351 nominal with elongated pad for handsoldering. (Body size source: IPC-SM-782 page 76, https://www.pcb-3d.com/wordpress/wp-content/uploads/ipc-sm-782a_amendment_1_and_2.pdf)")
+		(tags "capacitor handsolder")
 		(property "Reference" "C1"
-			(at 0 0.762 0)
+			(at 0 0.889 180)
 			(layer "F.SilkS")
 			(effects
 				(font
-					(size 0.6604 0.6604)
+					(size 0.8 0.8)
 					(thickness 0.15)
 				)
@@
 		)
 		(property "Value" "1uF"
-			(at 0 1.43 0)
+			(at 0 1.43 180)
 			(layer "F.Fab")
-			(hide yes)
 			(effects
 				(font
@@
 		)
 		(property "Datasheet" "~"
-			(at 0 0 0)
+			(at 0 0 180)
 			(layer "F.Fab")
 			(hide yes)
@@
 		)
 		(property "Description" ""
-			(at 0 0 0)
+			(at 0 0 180)
 			(layer "F.Fab")
 			(hide yes)
@@
 		(duplicate_pad_numbers_are_jumpers no)
 		(fp_line
-			(start -0.14058 0.51)
-			(end 0.14058 0.51)
+			(start -0.146267 0.51)
+			(end 0.146267 0.51)
 			(stroke
 				(width 0.12)
@@
 		)
 		(fp_line
-			(start -0.14058 -0.51)
-			(end 0.14058 -0.51)
+			(start -0.146267 -0.51)
+			(end 0.146267 -0.51)
 			(stroke
 				(width 0.12)
@@
 		)
 		(fp_rect
-			(start -1.48 -0.73)
-			(end 1.48 0.73)
+			(start -1.65 -0.73)
+			(end 1.65 0.73)
 			(stroke
 				(width 0.05)
@@
 		)
 		(fp_text user "${REFERENCE}"
-			(at 0 0 0)
+			(at 0 0 180)
 			(layer "F.Fab")
 			(effects
@@
 		)
 		(pad "1" smd roundrect
-			(at -0.775 0 180)
-			(size 0.9 0.95)
+			(at -0.8625 0 180)
+			(size 1.075 0.95)
 			(layers "F.Cu" "F.Mask" "F.Paste")
 			(roundrect_rratio 0.25)
@@
 		)
 		(pad "2" smd roundrect
-			(at 0.775 0 180)
-			(size 0.9 0.95)
+			(at 0.8625 0 180)
+			(size 1.075 0.95)
 			(layers "F.Cu" "F.Mask" "F.Paste")
 			(roundrect_rratio 0.25)
@@
 		)
 	)
-	(footprint "Resistor_SMD:R_0603_1608Metric"
+	(footprint "Resistor_SMD:R_0603_1608Metric_Pad0.98x0.95mm_HandSolder"
 		(layer "F.Cu")
 		(at 148.082 90.805 -90)
-		(descr "Resistor SMD 0603 (1608 Metric), square (rectangular) end terminal, IPC-7351 nominal, (Body size source: IPC-SM-782 page 72, https://www.pcb-3d.com/wordpress/wp-content/uploads/ipc-sm-782a_amendment_1_and_2.pdf)")
-		(tags "resistor")
+		(descr "Resistor SMD 0603 (1608 Metric), square (rectangular) end terminal, IPC-7351 nominal with elongated pad for handsoldering. (Body size source: IPC-SM-782 page 72, https://www.pcb-3d.com/wordpress/wp-content/uploads/ipc-sm-782a_amendment_1_and_2.pdf)")
+		(tags "resistor handsolder")
 		(property "Reference" "R2"
-			(at -2.286 0 90)
+			(at -2.54 0 270)
 			(layer "F.SilkS")
 			(effects
 				(font
-					(size 0.6604 0.6604)
+					(size 0.8 0.8)
 					(thickness 0.15)
 				)
@@
 		)
 		(property "Value" "4.7K"
-			(at 0 1.43 90)
+			(at 0 1.43 270)
 			(layer "F.Fab")
 			(effects
@@
 		)
 		(property "Datasheet" ""
-			(at 0 0 90)
+			(at 0 0 270)
 			(layer "F.Fab")
 			(hide yes)
@@
 		)
 		(property "Description" "Resistor"
-			(at 0 0 90)
+			(at 0 0 270)
 			(layer "F.Fab")
 			(hide yes)
@@
 		(duplicate_pad_numbers_are_jumpers no)
 		(fp_line
-			(start -0.237258 0.5225)
-			(end 0.237258 0.5225)
+			(start -0.254724 0.5225)
+			(end 0.254724 0.5225)
 			(stroke
 				(width 0.12)
@@
 		)
 		(fp_line
-			(start -0.237258 -0.5225)
-			(end 0.237258 -0.5225)
+			(start -0.254724 -0.5225)
+			(end 0.254724 -0.5225)
 			(stroke
 				(width 0.12)
@@
 		)
 		(fp_rect
-			(start -1.48 -0.73)
-			(end 1.48 0.73)
+			(start -1.65 -0.73)
+			(end 1.65 0.73)
 			(stroke
 				(width 0.05)
@@
 		)
 		(fp_text user "${REFERENCE}"
-			(at 0 0 90)
+			(at 0 0 270)
 			(layer "F.Fab")
 			(effects
@@
 		)
 		(pad "1" smd roundrect
-			(at -0.825 0 270)
-			(size 0.8 0.95)
+			(at -0.9125 0 270)
+			(size 0.975 0.95)
 			(layers "F.Cu" "F.Mask" "F.Paste")
 			(roundrect_rratio 0.25)
@@
 		)
 		(pad "2" smd roundrect
-			(at 0.825 0 270)
-			(size 0.8 0.95)
+			(at 0.9125 0 270)
+			(size 0.975 0.95)
 			(layers "F.Cu" "F.Mask" "F.Paste")
 			(roundrect_rratio 0.25)
@@
 			)
 		)
-		(property "Value" "LED"
+		(property "Value" "LED BLU"
 			(at -0.367 1.778 0)
 			(layer "F.Fab")
@@
 			)
 		)
-		(property "Value" "LED"
+		(property "Value" "LED GRN"
 			(at 0 1.43 0)
 			(layer "F.Fab")
@@
 	)
 	(segment
-		(start 148.082 99.708)
-		(end 148.323 99.949)
-		(width 0.4572)
-		(layer "F.Cu")
-		(net "+5V")
-	)
-	(segment
 		(start 145.044001 90.551)
 		(end 144.526 91.069001)
@@
 	)
 	(segment
+		(start 148.2355 99.949)
+		(end 146.825 99.949)
+		(width 0.4572)
+		(layer "F.Cu")
+		(net "+5V")
+	)
+	(segment
 		(start 148.092 97.165)
 		(end 148.102 97.155)
@@
 	)
 	(segment
+		(start 148.082 99.7955)
+		(end 148.2355 99.949)
+		(width 0.4572)
+		(layer "F.Cu")
+		(net "+5V")
+	)
+	(segment
 		(start 148.082 97.155)
-		(end 148.082 99.708)
+		(end 148.082 99.7955)
 		(width 0.4572)
 		(layer "F.Cu")
@@
 	)
 	(segment
-		(start 148.323 99.949)
-		(end 146.825 99.949)
-		(width 0.4572)
-		(layer "F.Cu")
-		(net "+5V")
-	)
-	(segment
 		(start 143.51 94.505)
 		(end 143.654 94.361)
@@
 	)
 	(segment
-		(start 145.2815 99.9425)
-		(end 145.275 99.949)
+		(start 145.542 99.682)
+		(end 145.2815 99.9425)
 		(width 0.4572)
 		(layer "F.Cu")
@@
 	)
 	(segment
-		(start 145.542 97.663)
-		(end 145.542 99.682)
+		(start 145.2815 99.9425)
+		(end 145.275 99.949)
 		(width 0.4572)
 		(layer "F.Cu")
@@
 	)
 	(segment
-		(start 145.542 99.682)
-		(end 145.2815 99.9425)
+		(start 145.542 97.663)
+		(end 145.542 99.682)
 		(width 0.4572)
 		(layer "F.Cu")

Commit message: Generate gerbers & fix C1/C2 overlapping courtyards
Parts:
- moved C2 0.25 mm to (149.4, 99.9)
Routing:
- net +5V: track 38.3 -> 39.2 mm
Changed lines of the file:
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@@
 			(outputformat 1)
 			(mirror no)
-			(drillshape 1)
+			(drillshape 0)
 			(scaleselection 1)
 			(outputdirectory "")
@@
 	(footprint "Capacitor_SMD:C_0603_1608Metric_Pad1.08x0.95mm_HandSolder"
 		(layer "F.Cu")
-		(at 149.098 99.949)
+		(at 149.352 99.949)
 		(descr "Capacitor SMD 0603 (1608 Metric), square (rectangular) end terminal, IPC-7351 nominal with elongated pad for handsoldering. (Body size source: IPC-SM-782 page 76, https://www.pcb-3d.com/wordpress/wp-content/uploads/ipc-sm-782a_amendment_1_and_2.pdf)")
 		(tags "capacitor handsolder")
@@
 	)
 	(segment
+		(start 148.4895 99.949)
+		(end 146.825 99.949)
+		(width 0.4572)
+		(layer "F.Cu")
+		(net "+5V")
+	)
+	(segment
 		(start 148.082 96.519)
 		(end 148.082 97.155)
@@
 	)
 	(segment
-		(start 148.2355 99.949)
-		(end 146.825 99.949)
-		(width 0.4572)
-		(layer "F.Cu")
-		(net "+5V")
-	)
-	(segment
 		(start 148.092 97.165)
 		(end 148.102 97.155)
@@
 	)
 	(segment
-		(start 148.082 99.7955)
-		(end 148.2355 99.949)
-		(width 0.4572)
-		(layer "F.Cu")
-		(net "+5V")
-	)
-	(segment
-		(start 148.082 97.155)
-		(end 148.082 99.7955)
+		(start 148.082 99.5415)
+		(end 148.4895 99.949)
 		(width 0.4572)
 		(layer "F.Cu")
@@
 		(width 0.4572)
 		(layer "F.Cu")
+		(net "+5V")
+	)
+	(segment
+		(start 148.082 96.6065)
+		(end 148.082 99.5415)
+		(width 0.4572)
+		(layer "F.Cu")
